Commit message: Renamed launch_config pkg to bringup as per best practices

File: anxious_robot_ws/src/robot_description/urdf/differential_drive_robot.xacro.urdf (robot description, URDF)
Before this commit: robot diff_bot, 2 links, 1 joints
Joints:
- joint caster_wheel_joint: origin xyz=-${caster_wheel_offset} 0 -${base_height / 2} rpy=0 0 0 -> xyz=-${caster_wheel_offset} 0.0 -${base_height / 2.0} rpy=0 0 0

Commit message: Connected base_footprint and base_link properly

File: anxious_robot_ws/src/robot_description/urdf/differential_drive_robot.xacro.urdf (robot description, URDF)
Before this commit: robot diff_bot, 3 links, 1 joints
Joints:
- added joint root_joint: type fixed, parent base_footprint, child base_link, origin xyz=0 0 0 rpy=0 0 0
