Commit message: Added front lidar links and joints to robot description

File: anxious_robot_ws/src/robot_description/urdf/properties.xacro (robot description, xacro)
@@ -9,3 +9,4 @@
     <xacro:property name="caster_wheel_radius" value="0.05" />
     <xacro:property name="caster_wheel_offset" value="0.1" />
+    <xacro:property name="front_lidar_arm_length" value="0.06" />
 </robot>

File: anxious_robot_ws/src/robot_description/urdf/sensors.xacro (robot description, xacro)
@@ -1,3 +1,47 @@
 <?xml version="1.0"?>
 <robot xmlns:xacro="http://www.ros.org/wiki/xacro" name="diff_bot">
+    <!-- <xacro:include filename="macros.xacro" />
+    <xacro:include filename="properties.xacro" /> -->
+    <link name="front_lidar_arm">
+        <xacro:box_inertia m="0.1" w="${front_lidar_arm_length}" h="0.02" d="0.02" />
+        <visual>
+            <origin xyz="0 0 0" rpy="0 0 0" />
+            <geometry>
+                <box size="${front_lidar_arm_length} 0.02 0.02" />
+            </geometry>
+            <!-- <material name="blue" /> -->
+        </visual>
+        <collision>
+            <origin xyz="0 0 0" rpy="0 0 0" />
+            <geometry>
+                <box size="${front_lidar_arm_length} 0.02 0.02" />
+            </geometry>
+        </collision>
+    </link>
+    <link name="front_lidar_link">
+        <xacro:box_inertia m="0.1" w="0.025" h="0.025" d="0.025" />
+        <visual>
+            <origin xyz="0 0 0" rpy="0 0 0" />
+            <geometry>
+                <box size="0.025 0.025 0.025" />
+            </geometry>
+            <!-- <material name="blue" /> -->
+        </visual>
+        <collision>
+            <origin xyz="0 0 0" rpy="0 0 0" />
+            <geometry>
+                <box size="0.025 0.025 0.025" />
+            </geometry>
+        </collision>
+    </link>
+    <joint name="front_lidar_arm_joint" type="fixed">
+        <parent link="base_link" />
+        <child link="front_lidar_arm" />
+        <origin xyz="${base_length/2 + front_lidar_arm_length/2} 0 0" rpy="0 0 0" />
+    </joint>
+    <joint name="front_lidar_joint" type="fixed">
+        <parent link="front_lidar_arm" />
+        <child link="front_lidar_link" />
+        <origin xyz="${front_lidar_arm_length/2 - 0.01} 0 -0.01" rpy="0 0 0" />
+    </joint>
 </robot>

Commit message: Applied cosmetic changes to robot description

File: anxious_robot_ws/src/robot_description/urdf/properties.xacro (robot description, xacro)
@@ -4,9 +4,10 @@
     <xacro:property name="base_length" value="0.4" />
     <xacro:property name="base_height" value="0.04" />
-    <xacro:property name="wheel_radius" value="0.07" />
+    <xacro:property name="wheel_radius" value="0.06" />
     <xacro:property name="wheel_length" value="0.01" />
     <xacro:property name="drive_wheel_offset" value="0.08" />
-    <xacro:property name="caster_wheel_radius" value="0.05" />
+    <xacro:property name="caster_wheel_radius" value="0.04" />
     <xacro:property name="caster_wheel_offset" value="0.1" />
     <xacro:property name="front_lidar_arm_length" value="0.06" />
+    <xacro:property name="front_lidar_size" value="0.015" />
 </robot>

File: anxious_robot_ws/src/robot_description/urdf/sensors.xacro (robot description, xacro)
@@ -20,9 +20,9 @@
     </link>
     <link name="front_lidar_link">
-        <xacro:box_inertia m="0.1" w="0.025" h="0.025" d="0.025" />
+        <xacro:box_inertia m="0.1" w="${front_lidar_size}" h="${front_lidar_size}" d="${front_lidar_size}" />
         <visual>
             <origin xyz="0 0 0" rpy="0 0 0" />
             <geometry>
-                <box size="0.025 0.025 0.025" />
+                <box size="${front_lidar_size} ${front_lidar_size} ${front_lidar_size}" />
             </geometry>
             <!-- <material name="blue" /> -->
@@ -31,5 +31,5 @@
             <origin xyz="0 0 0" rpy="0 0 0" />
             <geometry>
-                <box size="0.025 0.025 0.025" />
+                <box size="${front_lidar_size} ${front_lidar_size} ${front_lidar_size}" />
             </geometry>
         </collision>
