Commit message: Added gazebo references for front lidar links

File: anxious_robot_ws/src/robot_description/urdf/gazebo_elements.xacro (robot description, xacro)
@@ -12,4 +12,10 @@
     <gazebo reference="caster_wheel">
         <material>Gazebo/Yellow</material>
+    </gazebo>
+    <gazebo reference="front_lidar_arm">
+        <material>Gazebo/Blue</material>
+    </gazebo>
+    <gazebo reference="front_lidar_link">
+        <material>Gazebo/Green</material>
     </gazebo>
     <gazebo>

Commit message: Added front lidar sensor to robot description and applied further cosmetic changes

File: anxious_robot_ws/src/robot_description/urdf/gazebo_elements.xacro (robot description, xacro)
@@ -43,3 +43,37 @@
           </plugin>
     </gazebo>
+    <gazebo reference="front_lidar_link">
+        <sensor name="lidar" type="ray">
+            <always_on>true</always_on>
+            <visualize>true</visualize>
+            <update_rate>10</update_rate>
+            <ray>
+              <scan>
+                <vertical>
+                  <samples>1</samples>
+                  <resolution>1.000000</resolution>
+                  <min_angle>-1.570000</min_angle>
+                  <max_angle>-1.570001</max_angle>
+                </vertical>
+              </scan>
+              <range>
+                <min>0.010000</min>
+                <max>5</max>
+                <resolution>0.015000</resolution>
+              </range>
+              <noise>
+                <type>gaussian</type>
+                <mean>0.0</mean>
+                <stddev>0.01</stddev>
+              </noise>
+            </ray>
+            <plugin name="scan" filename="libgazebo_ros_ray_sensor.so">
+              <ros>
+                <remapping>~/out:=range</remapping>
+              </ros>
+              <output_type>sensor_msgs/Range</output_type>
+              <frame_name>lidar_link</frame_name>
+            </plugin>
+          </sensor>
+    </gazebo>
 </robot>

File: anxious_robot_ws/src/robot_description/urdf/properties.xacro (robot description, xacro)
@@ -10,4 +10,4 @@
     <xacro:property name="caster_wheel_offset" value="0.1" />
     <xacro:property name="front_lidar_arm_length" value="0.06" />
-    <xacro:property name="front_lidar_size" value="0.015" />
+    <xacro:property name="front_lidar_size" value="0.01" />
 </robot>

File: anxious_robot_ws/src/robot_description/urdf/sensors.xacro (robot description, xacro)
@@ -43,5 +43,5 @@
         <parent link="front_lidar_arm" />
         <child link="front_lidar_link" />
-        <origin xyz="${front_lidar_arm_length/2 - 0.01} 0 -0.01" rpy="0 0 0" />
+        <origin xyz="${front_lidar_arm_length/2 - front_lidar_size/2-0.002} 0 -${front_lidar_size}" rpy="0 0 0" />
     </joint>
 </robot>
